File: Mizuki_Power.kicad_blocks/PWR_Analog_1.kicad_block/PWR_Analog_1.kicad_sch (KiCad schematic)
At the start: 28 parts, among them Q1 AO3401A, Q2 AO3400A, U2 TPS62160DSG, U3 TLV61048DBVT, U4 SGM2209-5.0XN5G/TR, U5 TPS7A4701xRGW

Commit message: Corrected -5N EN level shifter
Parts:
- removed Q1: AO3401A, Package_TO_SOT_SMD:SOT-23, symbol Transistor_FET:AO3401A
- removed Q2: AO3400A, Package_TO_SOT_SMD:SOT-23, symbol Transistor_FET:AO3400A
- added Q1: AO3400A, Package_TO_SOT_SMD:SOT-23, symbol Transistor_FET:AO3400A
- added Q2: AO3401A, Package_TO_SOT_SMD:SOT-23, symbol Transistor_FET:AO3401A
- C?: renamed from C12; Part No. GRM188R61C106MA73# -> (none); Vendor muRata -> (none)
- renumbered C10 to C?, C8 to C?, C9 to C?, C11 to C?, C1 to C?, C5 to C?, C15 to C?, C13 to C?, C14 to C?, C2 to C?, C4 to C?, D1 to D?, D2 to D?, L1 to L?, L2 to L?, R8 to R?, R4 to R?, R5 to R?, R3 to R?, R7 to R?, R6 to R?, U4 to U?, U3 to U?, U5 to U?, U2 to U?
Connections:
- net GND: now also Q1.2 (S)
- net NEG_EN: now also Q2.3 (D)
- net OP_EN: now also Q1.1 (G)
- net VDC: now also Q2.2 (S)
- net at R?.2: now also Q1.3 (D), Q2.1 (G)
Other:
- note added: "+5V analog supply"
- note added: "-5V EN level shifter"
- note added: "-5V analog supply"
- moved on the sheet: C?, D?, L?, R?, U?
